File: hardware/servo.kicad_sch (KiCad schematic)
At the start: 40 parts, among them J1 5.5x2.1, J2 servo, J3 swd, J4 LED, Q1 DMT64M8LSS, SW1 restart, SW2 buzzer, U1 AOZ1284PI, U2 LDI1117-3.3U-DIO, U3 STM32G030F6Px

Commit message: Fix false stall detection after restart
Parts:
- J1: footprint Connector_BarrelJack:BarrelJack_diy -> Connector_BarrelJack:BarrelJack_GCT_DCJ200-10-A_Horizontal
Changed lines of the file:
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@@
 			)
 		)
-		(property "Footprint" "Connector_BarrelJack:BarrelJack_diy"
+		(property "Footprint" "Connector_BarrelJack:BarrelJack_GCT_DCJ200-10-A_Horizontal"
 			(at 12.7 21.336 0)
 			(hide yes)
