File: hardware/servo.kicad_sch (KiCad schematic)
At the start: 42 parts, among them J1 5.5x2.1, J2 servo, J3 swd, J4 LED, Q1 DMT64M8LSS, Q2 2N7000, SW1 restart, SW2 buzzer, U1 AOZ1284PI, U2 LDI1117-3.3U-DIO, U3 STM32G030F6Px

Commit message: Optimize buzzer, add beeping instead of steady tone
Parts:
- R10: value 3k -> 1k
- R9: value 1k -> 150
Changed lines of the file:
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@@
 			)
 		)
-		(property "Value" "3k"
+		(property "Value" "1k"
 			(at 167.64 54.6101 0)
 			(show_name no)
@@
 			)
 		)
-		(property "Value" "1k"
+		(property "Value" "150"
 			(at 153.67 45.7201 0)
 			(show_name no)

Commit message: Start project conversion to DC motor
Parts:
- removed C4: 4.7m, Capacitor_THT:CP_Radial_D16.0mm_P7.50mm, symbol Device:C_Polarized
- added R11: 220, Resistor_SMD:R_0805_2012Metric_Pad1.20x1.40mm_HandSolder, symbol Device:R
Connections:
- net fet: now also R11.2; no longer Q1.4 (G)
- net pwm: no longer names the net of J2.3 (Pin_3)
- net pwm: no longer U3.11 (PA4)
- new net: Q1.4 (G), R11.1
- no-connect marks 9 -> 11
Other:
- note added: "5v i 6v pakeist kompensacija pridetas r11, isimtas 4.7mf perdaryt korpusa?"
Changed lines of the file:
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@@
 	(generator_version "10.0")
 	(paper "A4")
+	(text "5v i 6v\npakeist kompensacija\npridetas r11, isimtas 4.7mf\nperdaryt korpusa?"
+		(exclude_from_sim no)
+		(at 183.388 85.852 0)
+		(effects
+			(font
+				(size 1.27 1.27)
+			)
+			(justify left)
+		)
+	)
 	(text "3khz"
 		(exclude_from_sim no)
@@
 	)
 	(junction
-		(at 238.76 22.86)
-		(diameter 0)
-		(color 0 0 0 0)
-	)
-	(junction
 		(at 119.38 29.21)
 		(diameter 0)
@@
 	)
 	(no_connect
+		(at 233.68 41.91)
+	)
+	(no_connect
 		(at 182.88 46.99)
 	)
@@
 	)
 	(no_connect
+		(at 273.05 26.67)
+	)
+	(no_connect
 		(at 233.68 39.37)
 	)
@@
 	(wire
 		(pts
-			(xy 67.31 19.05) (xy 71.12 19.05)
+			(xy 254 39.37) (xy 255.27 39.37)
 		)
 		(stroke
@@
 	(wire
 		(pts
-			(xy 266.7 29.21) (xy 273.05 29.21)
+			(xy 67.31 19.05) (xy 71.12 19.05)
 		)
 		(stroke
@@
 	(wire
 		(pts
-			(xy 111.76 29.21) (xy 119.38 29.21)
+			(xy 266.7 29.21) (xy 273.05 29.21)
 		)
 		(stroke
@@
 	(wire
 		(pts
-			(xy 273.05 26.67) (xy 269.24 26.67)
+			(xy 111.76 29.21) (xy 119.38 29.21)
 		)
 		(stroke
@@
 	(wire
 		(pts
-			(xy 245.11 39.37) (xy 255.27 39.37)
-		)
-		(stroke
-			(width 0)
-			(type default)
-		)
-	)
-	(wire
-		(pts
 			(xy 72.39 11.43) (xy 72.39 29.21)
 		)
@@
 	(wire
 		(pts
-			(xy 176.53 41.91) (xy 182.88 41.91)
+			(xy 245.11 39.37) (xy 246.38 39.37)
 		)
 		(stroke
@@
 	(wire
 		(pts
-			(xy 266.7 29.21) (xy 266.7 26.67)
+			(xy 176.53 41.91) (xy 182.88 41.91)
 		)
 		(stroke
@@
 	(wire
 		(pts
-			(xy 262.89 22.86) (xy 262.89 26.67)
+			(xy 266.7 29.21) (xy 266.7 26.67)
 		)
 		(stroke
@@
 	(wire
 		(pts
-			(xy 238.76 22.86) (xy 262.89 22.86)
-		)
-		(stroke
-			(width 0)
-			(type default)
-		)
-	)
-	(wire
-		(pts
 			(xy 66.04 52.07) (xy 66.04 57.15)
 		)
@@
 		)
 	)
-	(label "pwm"
-		(at 233.68 41.91 0)
-		(effects
-			(font
-				(size 1.27 1.27)
-			)
-			(justify left bottom)
-		)
-	)
-	(label "pwm"
-		(at 269.24 26.67 0)
-		(effects
-			(font
-				(size 1.27 1.27)
-			)
-			(justify left bottom)
-		)
-	)
 	(label "swclk"
 		(at 233.68 62.23 0)
@@
 	)
 	(symbol
-		(lib_id "Device:C_Polarized")
-		(at 238.76 26.67 0)
-		(mirror y)
-		(unit 1)
-		(body_style 1)
-		(exclude_from_sim no)
-		(in_bom yes)
-		(on_board yes)
-		(in_pos_files yes)
-		(dnp no)
-		(fields_autoplaced yes)
-		(property "Reference" "C4"
-			(at 242.57 24.5109 0)
-			(show_name no)
-			(do_not_autoplace no)
-			(effects
-				(font
-					(size 1.27 1.27)
-				)
-				(justify right)
-			)
-		)
-		(property "Value" "4.7m"
-			(at 242.57 27.0509 0)
-			(show_name no)
-			(do_not_autoplace no)
-			(effects
-				(font
-					(size 1.27 1.27)
-				)
-				(justify right)
-			)
-		)
-		(property "Footprint" "Capacitor_THT:CP_Radial_D16.0mm_P7.50mm"
-			(at 237.7948 30.48 0)
-			(hide yes)
-			(show_name no)
-			(do_not_autoplace no)
-			(effects
-				(font
-					(size 1.27 1.27)
-				)
-			)
-		)
-		(property "Datasheet" ""
-			(at 238.76 26.67 0)
-			(hide yes)
-			(show_name no)
-			(do_not_autoplace no)
-			(effects
-				(font
-					(size 1.27 1.27)
-				)
-			)
-		)
-		(property "Description" "Polarized capacitor"
-			(at 238.76 26.67 0)
-			(hide yes)
-			(show_name no)
-			(do_not_autoplace no)
-			(effects
-				(font
-					(size 1.27 1.27)
-				)
-			)
-		)
-		(pin "1"
-		)
-		(pin "2"
-		)
-		(instances
-			(project "servo"
-				(path "/868aa114-83f2-46f3-8e6d-8a7027303d9c"
-					(reference "C4")
-					(unit 1)
-				)
-			)
-		)
-	)
-	(symbol
 		(lib_id "Device:C")
 		(at 48.26 38.1 0)
@@
 	(symbol
 		(lib_id "power:GND")
-		(at 238.76 30.48 0)
-		(mirror y)
+		(at 67.31 26.67 0)
 		(unit 1)
 		(body_style 1)
@@
 		(dnp no)
 		(fields_autoplaced yes)
-		(property "Reference" "#PWR010"
-			(at 238.76 36.83 0)
+		(property "Reference" "#PWR07"
+			(at 67.31 33.02 0)
 			(hide yes)
 			(show_name no)
@@
 		)
 		(property "Value" "GND"
-			(at 238.76 35.56 0)
+			(at 67.31 31.75 0)
 			(show_name no)
 			(do_not_autoplace no)
@@
 		)
 		(property "Footprint" ""
-			(at 238.76 30.48 0)
+			(at 67.31 26.67 0)
 			(hide yes)
 			(show_name no)
@@
 		)
 		(property "Datasheet" ""
-			(at 238.76 30.48 0)
+			(at 67.31 26.67 0)
 			(hide yes)
 			(show_name no)
@@
 		)
 		(property "Description" "Power symbol creates a global label with name \"GND\" , ground"
-			(at 238.76 30.48 0)
+			(at 67.31 26.67 0)
 			(hide yes)
 			(show_name no)
@@
 			(project "servo"
 				(path "/868aa114-83f2-46f3-8e6d-8a7027303d9c"
-					(reference "#PWR010")
+					(reference "#PWR07")
 					(unit 1)
 				)
@@
 	)
 	(symbol
-		(lib_id "power:GND")
-		(at 67.31 26.67 0)
+		(lib_id "Device:L")
+		(at 107.95 29.21 90)
 		(unit 1)
 		(body_style 1)
@@
 		(dnp no)
 		(fields_autoplaced yes)
-		(property "Reference" "#PWR07"
-			(at 67.31 33.02 0)
-			(hide yes)
+		(property "Reference" "L1"
+			(at 107.95 24.13 90)
 			(show_name no)
 			(do_not_autoplace no)
@@
 			)
 		)
-		(property "Value" "GND"
-			(at 67.31 31.75 0)
+		(property "Value" "22u"
+			(at 107.95 26.67 90)
 			(show_name no)
 			(do_not_autoplace no)
@@
 			)
 		)
-		(property "Footprint" ""
-			(at 67.31 26.67 0)
+		(property "Footprint" "Inductor_SMD:LD2-HV"
+			(at 107.95 29.21 0)
 			(hide yes)
 			(show_name no)
@@
 		)
 		(property "Datasheet" ""
-			(at 67.31 26.67 0)
+			(at 107.95 29.21 0)
 			(hide yes)
 			(show_name no)
@@
 			)
 		)
-		(property "Description" "Power symbol creates a global label with name \"GND\" , ground"
-			(at 67.31 26.67 0)
+		(property "Description" "Inductor"
+			(at 107.95 29.21 0)
 			(hide yes)
 			(show_name no)
@@
 		(pin "1"
 		)
+		(pin "2"
+		)
 		(instances
 			(project "servo"
 				(path "/868aa114-83f2-46f3-8e6d-8a7027303d9c"
-					(reference "#PWR07")
+					(reference "L1")
 					(unit 1)
 				)
@@
 	)
 	(symbol
-		(lib_id "Device:L")
-		(at 107.95 29.21 90)
+		(lib_id "Device:R")
+		(at 250.19 39.37 270)
 		(unit 1)
 		(body_style 1)
@@
 		(in_pos_files yes)
 		(dnp no)
-		(fields_autoplaced yes)
-		(property "Reference" "L1"
-			(at 107.95 24.13 90)
+		(property "Reference" "R11"
+			(at 252.222 34.544 90)
 			(show_name no)
 			(do_not_autoplace no)
@@
 					(size 1.27 1.27)
 				)
+				(justify right)
 			)
 		)
-		(property "Value" "22u"
-			(at 107.95 26.67 90)
+		(property "Value" "220"
+			(at 252.222 37.084 90)
 			(show_name no)
 			(do_not_autoplace no)
@@
 					(size 1.27 1.27)
 				)
+				(justify right)
 			)
 		)
-		(property "Footprint" "Inductor_SMD:LD2-HV"
-			(at 107.95 29.21 0)
+		(property "Footprint" "Resistor_SMD:R_0805_2012Metric_Pad1.20x1.40mm_HandSolder"
+			(at 250.19 37.592 90)
 			(hide yes)
 			(show_name no)
@@
 		)
 		(property "Datasheet" ""
-			(at 107.95 29.21 0)
+			(at 250.19 39.37 0)
 			(hide yes)
 			(show_name no)
@@
 			)
 		)
-		(property "Description" "Inductor"
-			(at 107.95 29.21 0)
+		(property "Description" "Resistor"
+			(at 250.19 39.37 0)
 			(hide yes)
 			(show_name no)
@@
 			(project "servo"
 				(path "/868aa114-83f2-46f3-8e6d-8a7027303d9c"
-					(reference "L1")
+					(reference "R11")
 					(unit 1)
 				)
@@
 		(dnp no)
 		(property "Reference" "D1"
-			(at 259.842 29.972 90)
+			(at 259.842 26.162 90)
 			(show_name no)
 			(do_not_autoplace no)
@@
 		)
 		(property "Value" "SK310SMA"
-			(at 259.842 32.512 90)
+			(at 259.842 28.702 90)
 			(show_name no)
 			(do_not_autoplace no)
@@
 	(symbol
 		(lib_id "power:+5V")
-		(at 238.76 22.86 0)
+		(at 262.89 26.67 0)
 		(mirror y)
 		(unit 1)
@@
 		(fields_autoplaced yes)
 		(property "Reference" "#PWR08"
-			(at 238.76 26.67 0)
+			(at 262.89 30.48 0)
 			(hide yes)
 			(show_name no)
@@
 		)
 		(property "Value" "+5V"
-			(at 238.76 17.78 0)
+			(at 262.89 21.59 0)
 			(show_name no)
 			(do_not_autoplace no)
@@
 		)
 		(property "Footprint" ""
-			(at 238.76 22.86 0)
+			(at 262.89 26.67 0)
 			(hide yes)
 			(show_name no)
@@
 		)
 		(property "Datasheet" ""
-			(at 238.76 22.86 0)
+			(at 262.89 26.67 0)
 			(hide yes)
 			(show_name no)
@@
 		)
 		(property "Description" "Power symbol creates a global label with name \"+5V\""
-			(at 238.76 22.86 0)
+			(at 262.89 26.67 0)
 			(hide yes)
 			(show_name no)
