File: hardware/.history/servo.kicad_sch (KiCad schematic)
At the start: 42 parts, among them J1 5.5x2.1, J2 servo, J3 swd, J4 LED, Q1 DMT64M8LSS, Q2 2N7000, SW1 restart, SW2 buzzer, U1 AOZ1284PI, U2 LDI1117-3.3U-DIO, U3 STM32G030F6Px

Commit message: Add inductor parameters, add calculation file for 12V-6V conversion
Parts:
- R10: value 3k -> 1k
- R9: value 1k -> 150
Changed lines of the file:
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@@
 			)
 		)
-		(property "Value" "3k"
+		(property "Value" "1k"
 			(at 167.64 54.6101 0)
 			(show_name no)
@@
 			)
 		)
-		(property "Description" "Inductor"
+		(property "Description" "Inductor, 2A I_sat, 14.1u minimum"
 			(at 107.95 29.21 0)
 			(hide yes)
@@
 			)
 		)
-		(property "Value" "1k"
+		(property "Value" "150"
 			(at 153.67 45.7201 0)
 			(show_name no)
